File: Hardware/MM_MikroBUS_Carrier.brd (EAGLE design)
At the start: 85.1 x 35.6 mm, 106 parts, among them J15 MICROMOD-2222-C, J2 QWIIC_RIGHT_ANGLE, J5 Vertical Qwiic Connector, J7 MIKROBUS_SMD_BLACK1, J9 CORTEX_JTAG_DEBUG_MINIMUM_PTH, U1 MCP73831, U2 AP7361C-33FGEUDFN-8

Commit message: QC double-check
Routing:
- net VIN: track 78.2 -> 77.1 mm
Changed lines of the file:
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@@
 <drawing>
 <settings>
-<setting alwaysvectorfont="no"/>
+<setting alwaysvectorfont="yes"/>
 <setting verticaltext="up"/>
 </settings>
@@
 <wire x1="50.419" y1="7.366" x2="52.705" y2="5.08" width="0.4064" layer="16"/>
 <wire x1="52.705" y1="5.08" x2="52.705" y2="3.429" width="0.4064" layer="16"/>
-<wire x1="52.705" y1="3.429" x2="54.61" y2="1.524" width="0.4064" layer="16"/>
-<wire x1="54.61" y1="1.524" x2="59.69" y2="1.524" width="0.4064" layer="16"/>
-<via x="59.69" y="1.524" extent="1-16" drill="0.3048"/>
-<wire x1="59.69" y1="1.524" x2="59.69" y2="4.76" width="0.4064" layer="1"/>
+<wire x1="52.705" y1="3.429" x2="53.848" y2="2.286" width="0.4064" layer="16"/>
+<wire x1="53.848" y1="2.286" x2="59.69" y2="2.286" width="0.4064" layer="16"/>
+<via x="59.69" y="2.286" extent="1-16" drill="0.3048"/>
+<wire x1="59.69" y1="2.286" x2="59.69" y2="4.76" width="0.4064" layer="1"/>
 <wire x1="39.2049" y1="9.0551" x2="40.894" y2="7.366" width="0.4064" layer="16"/>
 </signal>

Commit message: Update MM_MikroBUS_Carrier.brd
Parts:
- removed U$20, U$21: (no value), output:#D1#0
- added U$19, U$6: (no value), output:#INT#0
- U$17, U$18: device output:#D0#0 -> output:#RST#0
- moved U$17 2.65 mm to (30.5, 29.7)
- moved U$18 2.65 mm to (30.5, 29.7)
Changed lines of the file:
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@@
 <?xml version="1.0" encoding="utf-8"?>
 <!DOCTYPE eagle SYSTEM "eagle.dtd">
-<eagle version="9.5.2">
+<eagle version="9.6.2">
 <drawing>
 <settings>
@@
 <element name="U$36" library="buzzard_labels (1)" package="#0" value="" x="1.143" y="17.399" smashed="yes"/>
 <element name="U$37" library="buzzard_labels (1)" package="#0" value="" x="7.366" y="23.495" smashed="yes"/>
-<element name="U$17" library="output" package="#D0#0" value="" x="33.02" y="30.48" smashed="yes" rot="R90"/>
-<element name="U$18" library="output" package="#D0#0" value="" x="33.02" y="30.48" smashed="yes" rot="MR90"/>
-<element name="U$20" library="output" package="#D1#0" value="" x="30.48" y="30.734" smashed="yes" rot="R90"/>
-<element name="U$21" library="output" package="#D1#0" value="" x="30.48" y="30.734" smashed="yes" rot="MR90"/>
 <element name="J6" library="SparkFun-Connectors" package="1X09_NO_SILK" value="" x="22.86" y="34.29" smashed="yes">
 <attribute name="NAME" x="21.59" y="35.687" size="0.6096" layer="25" font="vector" ratio="20"/>
@@
 <element name="U$38" library="output" package="#FUSEBYP#0" value="" x="15.367" y="21.59" smashed="yes" rot="MR0"/>
 <element name="U$39" library="output" package="#3V3EN#0" value="" x="15.748" y="16.51" smashed="yes" rot="MR0"/>
+<element name="U$6" library="output" package="#INT#0" value="" x="33.02" y="30.226" smashed="yes" rot="R90"/>
+<element name="U$19" library="output" package="#INT#0" value="" x="33.02" y="30.226" smashed="yes" rot="MR90"/>
+<element name="U$17" library="output" package="#RST#0" value="" x="30.48" y="29.718" smashed="yes" rot="R90"/>
+<element name="U$18" library="output" package="#RST#0" value="" x="30.48" y="29.718" smashed="yes" rot="MR90"/>
 </elements>
 <signals>
